File: synth_poly_vco_0.kicad_pcb (KiCad board)
At the start: 2 copper layers, 0 parts

Commit message: pcb layout
Parts:
- added C1: 1u, Capacitor_THT:CP_Radial_D6.3mm_P2.50mm, F.Cu at (-36.8, -125.7)
- added C10: 1u, Capacitor_THT:CP_Radial_D6.3mm_P2.50mm, F.Cu at (7.66, -88.9)
- added C11: 0.1u, Capacitor_THT:CP_Radial_D6.3mm_P2.50mm, F.Cu at (-3.81, -53.3)
- added C12: 1u, Capacitor_THT:CP_Radial_D6.3mm_P2.50mm, F.Cu at (-7.66, -97.8)
- added C2: 1u, Capacitor_THT:CP_Radial_D6.3mm_P2.50mm, F.Cu at (-36.8, -116.8)
- added C3: 0.1u, Capacitor_THT:CP_Radial_D6.3mm_P2.50mm, F.Cu at (-29.2, -125.7)
- added C4: 0.1u, Capacitor_THT:CP_Radial_D6.3mm_P2.50mm, F.Cu at (-29.2, -116.8)
- added C5: 0.1u, Capacitor_THT:CP_Radial_D6.3mm_P2.50mm, F.Cu at (-3.81, -76.2)
- added C6: 0.1u, Capacitor_THT:CP_Radial_D6.3mm_P2.50mm, F.Cu at (-3.81, -68.5)
- added C7: 2.2n, Capacitor_THT:CP_Radial_D6.3mm_P2.50mm, F.Cu at (-3.81, -60.9)
- added C8: 0.1u, Capacitor_THT:CP_Radial_D6.3mm_P2.50mm, F.Cu at (22.8, -104.1)
- added C9: 0.1u, Capacitor_THT:CP_Radial_D6.3mm_P2.50mm, F.Cu at (22.8, -114.3)
- added D1: 1N5819, Diode_THT:D_DO-41_SOD81_P10.16mm_Horizontal, F.Cu at (-29.0, -96.0)
- added D2: 1N5819, Diode_THT:D_DO-41_SOD81_P10.16mm_Horizontal, F.Cu at (-25.2, -106.2)
- added D3: 1N4148WS, Diode_SMD:D_SOD-323, F.Cu at (5.08, -59.9)
- added D4: 1N4148WS, Diode_SMD:D_SOD-323, F.Cu at (0.64, -105.2)
- added D5: 1N4148WS, Diode_SMD:D_SOD-323, F.Cu at (-3.17, -105.2)
- added J1: Power, Connector_IDC:IDC-Header_2x07-1MP_P2.54mm_Latch_Vertical, F.Cu at (-10.2, -125.7)
- added J2: IN_vco, Connector_PinHeader_2.54mm:PinHeader_1x02_P2.54mm_Vertical, F.Cu at (-36.8, -57.1)
- added J3: Conn_01x02_Pin, Connector_PinHeader_2.54mm:PinHeader_1x02_P2.54mm_Vertical, F.Cu at (-17.8, -77.5)
- added J4: OUT_triangle, Connector_PinHeader_2.54mm:PinHeader_1x02_P2.54mm_Vertical, F.Cu at (-17.8, -100.3)
- added J5: OUT_saw, Connector_PinHeader_2.54mm:PinHeader_1x02_P2.54mm_Vertical, F.Cu at (25.4, -48.3)
- added J6: OUT_pwm, Connector_PinHeader_2.54mm:PinHeader_1x02_P2.54mm_Vertical, F.Cu at (26.7, -91.4)
- added Q1: BC558, Package_TO_SOT_THT:TO-92_Inline, F.Cu at (-22.9, -58.4)
- added Q2: BC548, Package_TO_SOT_THT:TO-92_Inline, F.Cu at (-17.8, -61.0)
- added R1: 100k, Resistor_THT:R_Axial_DIN0204_L3.6mm_D1.6mm_P7.62mm_Horizontal, F.Cu at (-31.7, -88.9)
- added R10: 1M, Resistor_THT:R_Axial_DIN0204_L3.6mm_D1.6mm_P7.62mm_Horizontal, F.Cu at (-12.7, -50.8)
- added R11: 68k, Resistor_THT:R_Axial_DIN0204_L3.6mm_D1.6mm_P7.62mm_Horizontal, F.Cu at (-1.27, -81.3)
- added R12: 100k, Resistor_THT:R_Axial_DIN0204_L3.6mm_D1.6mm_P7.62mm_Horizontal, F.Cu at (-6.35, -81.3)
- added R13: 100k, Resistor_THT:R_Axial_DIN0204_L3.6mm_D1.6mm_P7.62mm_Horizontal, F.Cu at (19.1, -80.0)
- added R14: 14k, Resistor_THT:R_Axial_DIN0204_L3.6mm_D1.6mm_P7.62mm_Horizontal, F.Cu at (-3.81, -88.9)
- added R15: 100k, Resistor_THT:R_Axial_DIN0204_L3.6mm_D1.6mm_P7.62mm_Horizontal, F.Cu at (22.9, -63.5)
- added R16: 47k, Resistor_THT:R_Axial_DIN0204_L3.6mm_D1.6mm_P7.62mm_Horizontal, F.Cu at (20.3, -63.5)
- added R17: 100k, Resistor_THT:R_Axial_DIN0204_L3.6mm_D1.6mm_P7.62mm_Horizontal, F.Cu at (24.1, -69.8)
- added R18: 50k, Resistor_THT:R_Axial_DIN0204_L3.6mm_D1.6mm_P7.62mm_Horizontal, F.Cu at (-6.99, -116.8)
- added R19: 60k, Resistor_THT:R_Axial_DIN0204_L3.6mm_D1.6mm_P7.62mm_Horizontal, F.Cu at (26.7, -77.5)
- added R2: 33k, Resistor_THT:R_Axial_DIN0204_L3.6mm_D1.6mm_P7.62mm_Horizontal, F.Cu at (-34.2, -88.9)
- added R20: 50k, Resistor_THT:R_Axial_DIN0204_L3.6mm_D1.6mm_P7.62mm_Horizontal, F.Cu at (-4.45, -109.2)
- added R21: 20k, Resistor_THT:R_Axial_DIN0204_L3.6mm_D1.6mm_P7.62mm_Horizontal, F.Cu at (-1.91, -109.2)
- added R22: 200k, Resistor_THT:R_Axial_DIN0204_L3.6mm_D1.6mm_P7.62mm_Horizontal, F.Cu at (-14.0, -97.8)
- added R23: 1k, Resistor_THT:R_Axial_DIN0204_L3.6mm_D1.6mm_P7.62mm_Horizontal, F.Cu at (25.4, -63.5)
- added R24: 1k, Resistor_THT:R_Axial_DIN0204_L3.6mm_D1.6mm_P7.62mm_Horizontal, F.Cu at (19.1, -90.2)
- added R3: 100k, Resistor_THT:R_Axial_DIN0204_L3.6mm_D1.6mm_P7.62mm_Horizontal, F.Cu at (-33.0, -73.7)
- added R4: 100k, Resistor_THT:R_Axial_DIN0204_L3.6mm_D1.6mm_P7.62mm_Horizontal, F.Cu at (-29.1, -88.9)
- added R5: 1M, Resistor_THT:R_Axial_DIN0204_L3.6mm_D1.6mm_P7.62mm_Horizontal, F.Cu at (-30.5, -66.0)
- added R6: 10, Resistor_THT:R_Axial_DIN0204_L3.6mm_D1.6mm_P7.62mm_Horizontal, F.Cu at (-37.6, -97.3)
- added R7: 10, Resistor_THT:R_Axial_DIN0204_L3.6mm_D1.6mm_P7.62mm_Horizontal, F.Cu at (-34.1, -97.3)
- added R8: 100k, Resistor_THT:R_Axial_DIN0204_L3.6mm_D1.6mm_P7.62mm_Horizontal, F.Cu at (-33.0, -54.6)
- added R9: 1.5K, Resistor_THT:R_Axial_DIN0204_L3.6mm_D1.6mm_P7.62mm_Horizontal, F.Cu at (-33.0, -49.5)
- added RV1: 100k, Potentiometer_THT:Potentiometer_Bourns_3266Y_Vertical, F.Cu at (-38.1, -87.6)
- added RV2: 100k, Potentiometer_THT:Potentiometer_Bourns_3266Y_Vertical, F.Cu at (-36.8, -72.4)
- added RV3: 1k, Potentiometer_THT:Potentiometer_Bourns_3266Y_Vertical, F.Cu at (-36.8, -48.3)
- added RV4: 100k, Potentiometer_THT:Potentiometer_Bourns_3266Y_Vertical, F.Cu at (-11.4, -78.7)
- added RV5: 100k, Potentiometer_THT:Potentiometer_Bourns_3266Y_Vertical, F.Cu at (-11.4, -87.6)
- added RV6: 100k, Potentiometer_THT:Potentiometer_Bourns_3266Y_Vertical, F.Cu at (-10.8, -115.6)
- added TH1: NTC 10k, Resistor_THT:R_Axial_DIN0204_L3.6mm_D1.6mm_P2.54mm_Vertical, F.Cu at (-25.4, -86.4)
- added TH2: NTC 10k, Resistor_THT:R_Axial_DIN0204_L3.6mm_D1.6mm_P2.54mm_Vertical, F.Cu at (-27.9, -71.1)
- added TP1: TestPoint, TestPoint:TestPoint_Pad_D1.5mm, F.Cu at (-24.1, -52.1)
- added TP2: TestPoint, TestPoint:TestPoint_Pad_D1.5mm, F.Cu at (1.27, -52.1)
- added TP3: TestPoint, TestPoint:TestPoint_Pad_D1.5mm, F.Cu at (21.6, -74.9)
- added TP4: TestPoint, TestPoint:TestPoint_Pad_D1.5mm, F.Cu at (-1.27, -95.2)
- added TP5: TestPoint, TestPoint:TestPoint_Pad_D1.5mm, F.Cu at (24.1, -82.5)
- added TP6: TestPoint, TestPoint:TestPoint_Pad_D1.5mm, F.Cu at (-15.9, -110.5)
- added TP7: TestPoint, TestPoint:TestPoint_Pad_D1.5mm, F.Cu at (3.17, -110.5)
- added U1: TL074, Package_DIP:DIP-14_W7.62mm_Socket, F.Cu at (7.62, -82.5)
- added U2: 40106, Package_DIP:DIP-14_W7.62mm_Socket, F.Cu at (7.62, -61.0)
- added U3: TL072, Package_DIP:DIP-14_W7.62mm_Socket, F.Cu at (7.62, -116.2)
Routing:
- net -12V: track 0.00 -> 310.6 mm
- net +12V: track 0.00 -> 192.7 mm
- net Net-(U1C--): track 0.00 -> 72.4 mm
- net Net-(D3-K): track 0.00 -> 53.5 mm
- net Net-(Q1-B): track 0.00 -> 52.2 mm
- net Net-(D1-A): track 0.00 -> 45.4 mm
- net Net-(U1B-+): track 0.00 -> 31.5 mm
- net Net-(D2-K): track 0.00 -> 28.3 mm
- net Net-(D4-K): track 0.00 -> 27.0 mm
- net Net-(D5-A): track 0.00 -> 27.0 mm
- net Net-(D4-A): track 0.00 -> 26.2 mm
- net Net-(R15-Pad2): track 0.00 -> 22.5 mm
- net Net-(U1B--): track 0.00 -> 17.9 mm
- net Net-(J5-Pin_1): track 0.00 -> 16.5 mm
- net Net-(U1D-+): track 0.00 -> 16.5 mm
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
Commit message: modify icd optimized paths add descriptions to in and outputs
Parts:
- added TP10: Test Point, TestPoint:TestPoint_Pad_D1.5mm, F.Cu at (135.9, 134.6)
- added TP11: Test Point, TestPoint:TestPoint_Pad_D1.5mm, F.Cu at (176.5, 67.3)
- added TP8: TestPoint, TestPoint:TestPoint_Pad_D1.5mm, F.Cu at (149.9, 130.8)
- added TP9: TestPoint, TestPoint:TestPoint_Pad_D1.5mm, F.Cu at (168.9, 94.0)
- D3, D4, D5: value 1N4148WS -> 1N4148; footprint Diode_SMD:D_SOD-323 -> Diode_THT:D_DO-35_SOD27_P7.62mm_Horizontal
- J1: value Power -> Conn_02x08_Odd_Even; footprint Connector_IDC:IDC-Header_2x07-1MP_P2.54mm_Latch_Vertical -> Connector_IDC:IDC-Header_2x08_P2.54mm_Vertical; moved to B.Cu
- R11: value 68k -> 100k
- R12: value 100k -> 68k
- TP1, TP2, TP3, TP4, TP5, TP6, TP7: value TestPoint -> Test Point
- U3: footprint Package_DIP:DIP-14_W7.62mm_Socket -> Package_DIP:DIP-8_W7.62mm_Socket
- moved J4 266.1 mm to (179.1, 78.7), turned to 90 degrees
- moved R14 261.6 mm to (132.1, 134.6), turned to 180 degrees
- moved R21 260.5 mm to (170.2, 86.4), turned to 180 degrees
- moved C3 256.0 mm to (154.9, 52.1)
- moved C4 255.9 mm to (154.9, 61.0)
- moved C5 255.1 mm to (153.7, 124.5)
- moved C1 255.1 mm to (146.1, 52.1)
- moved C2 255.1 mm to (146.1, 61.0)
- moved C6 254.8 mm to (162.6, 124.5)
- moved RV5 254.3 mm to (116.8, 132.0), turned to 0 degrees
- moved R22 253.3 mm to (162.6, 83.8), turned to 0 degrees
- moved J2 253.0 mm to (115.6, 144.8), turned to -90 degrees
- moved C7 251.4 mm to (146.1, 141.0)
- moved D5 251.1 mm to (182.9, 63.5), turned to 90 degrees
- moved R24 251.1 mm to (176.5, 105.4), turned to 180 degrees
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Connections:
- net Net-(D1-A) renamed +12V_raw
- net Net-(D2-K) renamed -12V_raw
- J1 pad 13: unconnected-(J1-Pin_13-Pad13) -> CV
- J1 pad 14: unconnected-(J1-Pin_14-Pad14) -> CV
- R11 pad 1: Net-(R11-Pad1) -> GND
- R11 pad 2: Net-(U1C--) -> Net-(U1B-+)
- R13 pad 1: GND -> Net-(R13-Pad1)
- R13 pad 2: Net-(U1B-+) -> Net-(U1C--)
- RV4 pad 2: Net-(R11-Pad1) -> Net-(R12-Pad1)
- RV4 pad 3: Net-(R11-Pad1) -> Net-(R12-Pad1)
- RV5 pad 2: Net-(R12-Pad1) -> Net-(R13-Pad1)
- TP1 pad 1: Net-(Q1-B) -> Gate
- TP2 pad 1: Net-(D3-K) -> CV
- TP3 pad 1: Net-(U1B-+) -> +5V
- TP4 pad 1: Net-(U1C--) -> +12V
- TP5 pad 1: Net-(U1D-+) -> GND
- TP6 pad 1: Net-(U3B--) -> -12V
- TP7 pad 1: Net-(D4-K) -> Net-(Q1-B)
Routing:
- net Net-(U3B--): track 5.08 -> 79.1 mm
- net Net-(U1B-+): track 31.5 -> 86.0 mm
- net Net-(J2-Pin_1): track 5.61 -> 59.2 mm
- net -12V: track 310.6 -> 259.4 mm
- net -12V_raw: track 28.3 -> 67.9 mm
- net Net-(D5-A): track 27.0 -> 63.2 mm
- net Net-(D4-A): track 26.2 -> 57.6 mm
- net Net-(J4-Pin_1): track 8.67 -> 38.6 mm
- net Net-(U1C--): track 72.4 -> 48.3 mm
- net +12V: track 192.7 -> 215.8 mm
- net Net-(D4-K): track 27.0 -> 49.8 mm
- net Net-(Q1-B): track 52.2 -> 35.6 mm
- net Net-(R11-Pad1): track 14.8 -> 0.00 mm
- net Net-(U1A--): track 8.91 -> 22.8 mm
- net Net-(R13-Pad1): track 0.00 -> 12.3 mm
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- added copper zone on B.Cu, net GND
- added copper zone on F.Cu, net GND
Other:
- board outline added: 77.5 x 129.5 mm
